File: AutoRouter/output.kicad_pcb (KiCad board)
At the start: 2 copper layers, 104 x 83.9 mm, 30 parts

Commit message: adjusted autorouter timing, added switch referencing
Parts:
- removed ADC1: TLA2528IRTER, TLA2528IRTER:WQFN16_RTE_TEX
- removed C1, C2: 2uF, Capacitor_SMD:C_0805_2012Metric_Pad1.18x1.45mm_HandSolder
- removed H1, H10, H11, H12, H13, H14, H15, H16, H2, H3, H4, H5, H6, H7, H8, H9: AH49FNTR-G1, AH49FNTR_G1:SC59_DIO_KeyswitchOutline_NoRuleArea
- removed MCU1: RP2040-Zero, RP2040-Zero:rp2040-zero-tht
- removed Sensor_Driver1: TLC59108IRGYR, TLC59208FIRGYR:RGY16_2P55X2P05
- removed TP1: col0, TestPoint:TestPoint_Pad_2.0x2.0mm
- removed TP2: col1, TestPoint:TestPoint_Pad_2.0x2.0mm
- removed TP3: col2, TestPoint:TestPoint_Pad_2.0x2.0mm
- removed TP4: col3, TestPoint:TestPoint_Pad_2.0x2.0mm
- removed TP5: row0, TestPoint:TestPoint_Pad_2.0x2.0mm
- removed TP6: row1, TestPoint:TestPoint_Pad_2.0x2.0mm
- removed TP7: row2, TestPoint:TestPoint_Pad_2.0x2.0mm
- removed TP8: row3, TestPoint:TestPoint_Pad_2.0x2.0mm
- removed TP9: GND, TestPoint:TestPoint_Pad_2.0x2.0mm
- added SW1: SC59_DIO_KeyswitchOutline_NoRuleArea_mosfet, SC59_DIO_KeyswitchOutline_NoRuleArea_mosfet, F.Cu at (9.53, 9.53)
- added SW10: SC59_DIO_KeyswitchOutline_NoRuleArea_mosfet, SC59_DIO_KeyswitchOutline_NoRuleArea, F.Cu at (181.0, 9.53)
- added SW11: SC59_DIO_KeyswitchOutline_NoRuleArea_mosfet, SC59_DIO_KeyswitchOutline_NoRuleArea, F.Cu at (200.0, 9.53)
- added SW12: SC59_DIO_KeyswitchOutline_NoRuleArea_mosfet, SC59_DIO_KeyswitchOutline_NoRuleArea, F.Cu at (219.1, 9.53)
- added SW13: SC59_DIO_KeyswitchOutline_NoRuleArea_mosfet, SC59_DIO_KeyswitchOutline_NoRuleArea, F.Cu at (238.1, 9.53)
- added SW14: SC59_DIO_KeyswitchOutline_NoRuleArea_mosfet, SC59_DIO_KeyswitchOutline_NoRuleArea, F.Cu at (257.2, 9.53)
- added SW15: SC59_DIO_KeyswitchOutline_NoRuleArea_mosfet, SC59_DIO_KeyswitchOutline_NoRuleArea, F.Cu at (9.53, 28.6)
- added SW16: SC59_DIO_KeyswitchOutline_NoRuleArea_mosfet, SC59_DIO_KeyswitchOutline_NoRuleArea, F.Cu at (33.3, 28.6)
- added SW17: SC59_DIO_KeyswitchOutline_NoRuleArea_mosfet, SC59_DIO_KeyswitchOutline_NoRuleArea_mosfet, F.Cu at (52.4, 28.6)
- added SW18: SC59_DIO_KeyswitchOutline_NoRuleArea_mosfet, SC59_DIO_KeyswitchOutline_NoRuleArea, F.Cu at (71.4, 28.6)
- added SW19: SC59_DIO_KeyswitchOutline_NoRuleArea_mosfet, SC59_DIO_KeyswitchOutline_NoRuleArea, F.Cu at (90.5, 28.6)
- added SW2: SC59_DIO_KeyswitchOutline_NoRuleArea_mosfet, SC59_DIO_KeyswitchOutline_NoRuleArea, F.Cu at (28.6, 9.53)
- added SW20: SC59_DIO_KeyswitchOutline_NoRuleArea_mosfet, SC59_DIO_KeyswitchOutline_NoRuleArea, F.Cu at (109.5, 28.6)
- added SW21: SC59_DIO_KeyswitchOutline_NoRuleArea_mosfet, SC59_DIO_KeyswitchOutline_NoRuleArea, F.Cu at (128.6, 28.6)
- added SW22: SC59_DIO_KeyswitchOutline_NoRuleArea_mosfet, SC59_DIO_KeyswitchOutline_NoRuleArea, F.Cu at (147.6, 28.6)
- added SW23: SC59_DIO_KeyswitchOutline_NoRuleArea_mosfet, SC59_DIO_KeyswitchOutline_NoRuleArea, F.Cu at (166.7, 28.6)
- added SW24: SC59_DIO_KeyswitchOutline_NoRuleArea_mosfet, SC59_DIO_KeyswitchOutline_NoRuleArea, F.Cu at (185.7, 28.6)
- added SW25: SC59_DIO_KeyswitchOutline_NoRuleArea_mosfet, SC59_DIO_KeyswitchOutline_NoRuleArea_mosfet, F.Cu at (204.8, 28.6)
- added SW26: SC59_DIO_KeyswitchOutline_NoRuleArea_mosfet, SC59_DIO_KeyswitchOutline_NoRuleArea, F.Cu at (223.8, 28.6)
- added SW27: SC59_DIO_KeyswitchOutline_NoRuleArea_mosfet, SC59_DIO_KeyswitchOutline_NoRuleArea, F.Cu at (242.9, 28.6)
- added SW28: SC59_DIO_KeyswitchOutline_NoRuleArea_mosfet, SC59_DIO_KeyswitchOutline_NoRuleArea, F.Cu at (261.9, 28.6)
- added SW29: SC59_DIO_KeyswitchOutline_NoRuleArea_mosfet, SC59_DIO_KeyswitchOutline_NoRuleArea, F.Cu at (9.53, 47.6)
- added SW3: SC59_DIO_KeyswitchOutline_NoRuleArea_mosfet, SC59_DIO_KeyswitchOutline_NoRuleArea, F.Cu at (47.6, 9.53)
- added SW30: SC59_DIO_KeyswitchOutline_NoRuleArea_mosfet, SC59_DIO_KeyswitchOutline_NoRuleArea, F.Cu at (38.1, 47.6)
- added SW31: SC59_DIO_KeyswitchOutline_NoRuleArea_mosfet, SC59_DIO_KeyswitchOutline_NoRuleArea, F.Cu at (57.1, 47.6)
- added SW32: SC59_DIO_KeyswitchOutline_NoRuleArea_mosfet, SC59_DIO_KeyswitchOutline_NoRuleArea, F.Cu at (76.2, 47.6)
- added SW33: SC59_DIO_KeyswitchOutline_NoRuleArea_mosfet, SC59_DIO_KeyswitchOutline_NoRuleArea_mosfet, F.Cu at (95.2, 47.6)
- added SW34: SC59_DIO_KeyswitchOutline_NoRuleArea_mosfet, SC59_DIO_KeyswitchOutline_NoRuleArea, F.Cu at (114.3, 47.6)
- added SW35: SC59_DIO_KeyswitchOutline_NoRuleArea_mosfet, SC59_DIO_KeyswitchOutline_NoRuleArea, F.Cu at (133.3, 47.6)
- added SW36: SC59_DIO_KeyswitchOutline_NoRuleArea_mosfet, SC59_DIO_KeyswitchOutline_NoRuleArea, F.Cu at (152.4, 47.6)
- added SW37: SC59_DIO_KeyswitchOutline_NoRuleArea_mosfet, SC59_DIO_KeyswitchOutline_NoRuleArea, F.Cu at (171.4, 47.6)
- added SW38: SC59_DIO_KeyswitchOutline_NoRuleArea_mosfet, SC59_DIO_KeyswitchOutline_NoRuleArea, F.Cu at (190.5, 47.6)
- added SW39: SC59_DIO_KeyswitchOutline_NoRuleArea_mosfet, SC59_DIO_KeyswitchOutline_NoRuleArea, F.Cu at (209.6, 47.6)
- added SW4: SC59_DIO_KeyswitchOutline_NoRuleArea_mosfet, SC59_DIO_KeyswitchOutline_NoRuleArea, F.Cu at (66.7, 9.53)
- added SW40: SC59_DIO_KeyswitchOutline_NoRuleArea_mosfet, SC59_DIO_KeyswitchOutline_NoRuleArea, F.Cu at (228.6, 47.6)
- added SW41: SC59_DIO_KeyswitchOutline_NoRuleArea_mosfet, SC59_DIO_KeyswitchOutline_NoRuleArea_mosfet, F.Cu at (247.7, 47.6)
- added SW42: SC59_DIO_KeyswitchOutline_NoRuleArea_mosfet, SC59_DIO_KeyswitchOutline_NoRuleArea, F.Cu at (9.53, 66.7)
- added SW43: SC59_DIO_KeyswitchOutline_NoRuleArea_mosfet, SC59_DIO_KeyswitchOutline_NoRuleArea, F.Cu at (42.9, 66.7)
- added SW44: SC59_DIO_KeyswitchOutline_NoRuleArea_mosfet, SC59_DIO_KeyswitchOutline_NoRuleArea, F.Cu at (61.9, 66.7)
- added SW45: SC59_DIO_KeyswitchOutline_NoRuleArea_mosfet, SC59_DIO_KeyswitchOutline_NoRuleArea, F.Cu at (81.0, 66.7)
- added SW46: SC59_DIO_KeyswitchOutline_NoRuleArea_mosfet, SC59_DIO_KeyswitchOutline_NoRuleArea, F.Cu at (100.0, 66.7)
- added SW47: SC59_DIO_KeyswitchOutline_NoRuleArea_mosfet, SC59_DIO_KeyswitchOutline_NoRuleArea, F.Cu at (119.1, 66.7)
- added SW48: SC59_DIO_KeyswitchOutline_NoRuleArea_mosfet, SC59_DIO_KeyswitchOutline_NoRuleArea, F.Cu at (138.1, 66.7)
- added SW49: SC59_DIO_KeyswitchOutline_NoRuleArea_mosfet, SC59_DIO_KeyswitchOutline_NoRuleArea_mosfet, F.Cu at (157.2, 66.7)
- added SW5: SC59_DIO_KeyswitchOutline_NoRuleArea_mosfet, SC59_DIO_KeyswitchOutline_NoRuleArea, F.Cu at (85.7, 9.53)
- added SW50: SC59_DIO_KeyswitchOutline_NoRuleArea_mosfet, SC59_DIO_KeyswitchOutline_NoRuleArea, F.Cu at (176.2, 66.7)
- added SW51: SC59_DIO_KeyswitchOutline_NoRuleArea_mosfet, SC59_DIO_KeyswitchOutline_NoRuleArea, F.Cu at (195.3, 66.7)
- added SW52: SC59_DIO_KeyswitchOutline_NoRuleArea_mosfet, SC59_DIO_KeyswitchOutline_NoRuleArea, F.Cu at (214.3, 66.7)
- added SW53: SC59_DIO_KeyswitchOutline_NoRuleArea_mosfet, SC59_DIO_KeyswitchOutline_NoRuleArea, F.Cu at (233.4, 66.7)
- added SW54: SC59_DIO_KeyswitchOutline_NoRuleArea_mosfet, SC59_DIO_KeyswitchOutline_NoRuleArea, F.Cu at (9.53, 85.7)
- added SW55: SC59_DIO_KeyswitchOutline_NoRuleArea_mosfet, SC59_DIO_KeyswitchOutline_NoRuleArea, F.Cu at (33.3, 85.7)
- added SW56: SC59_DIO_KeyswitchOutline_NoRuleArea_mosfet, SC59_DIO_KeyswitchOutline_NoRuleArea, F.Cu at (52.4, 85.7)
- added SW57: SC59_DIO_KeyswitchOutline_NoRuleArea_mosfet, SC59_DIO_KeyswitchOutline_NoRuleArea_mosfet, F.Cu at (76.2, 85.7)
- added SW58: SC59_DIO_KeyswitchOutline_NoRuleArea_mosfet, SC59_DIO_KeyswitchOutline_NoRuleArea, F.Cu at (195.3, 85.7)
- added SW59: SC59_DIO_KeyswitchOutline_NoRuleArea_mosfet, SC59_DIO_KeyswitchOutline_NoRuleArea, F.Cu at (219.1, 85.7)
- added SW6: SC59_DIO_KeyswitchOutline_NoRuleArea_mosfet, SC59_DIO_KeyswitchOutline_NoRuleArea, F.Cu at (104.8, 9.53)
- added SW60: SC59_DIO_KeyswitchOutline_NoRuleArea_mosfet, SC59_DIO_KeyswitchOutline_NoRuleArea, F.Cu at (238.1, 85.7)
- added SW61: SC59_DIO_KeyswitchOutline_NoRuleArea_mosfet, SC59_DIO_KeyswitchOutline_NoRuleArea, F.Cu at (257.2, 85.7)
- added SW62: WQFN16_RTE_TEX_with_caps_and_Rs, WQFN16_RTE_TEX_with_caps_and_Rs, F.Cu at (21.0, 21.0)
- added SW63: WQFN16_RTE_TEX_with_caps_and_Rs, WQFN16_RTE_TEX_with_caps_and_Rs, F.Cu at (21.0, 32.4)
- added SW7: SC59_DIO_KeyswitchOutline_NoRuleArea_mosfet, SC59_DIO_KeyswitchOutline_NoRuleArea, F.Cu at (123.8, 9.53)
- added SW8: SC59_DIO_KeyswitchOutline_NoRuleArea_mosfet, SC59_DIO_KeyswitchOutline_NoRuleArea, F.Cu at (142.9, 9.53)
- added SW9: SC59_DIO_KeyswitchOutline_NoRuleArea_mosfet, SC59_DIO_KeyswitchOutline_NoRuleArea_mosfet, F.Cu at (161.9, 9.53)
- added U?: rp2040-zero-tht, rp2040-zero-tht, F.Cu at (305.7, 12.8)
Routing:
- net GND: track 354.0 -> 626.4 mm
- net m0c2: track 0.00 -> 267.8 mm, vias 0 -> 5
- net +3.3v: track 0.00 -> 242.8 mm, vias 0 -> 3
- net m0r7MOS: track 0.00 -> 186.1 mm, vias 0 -> 2
- net m0r3: track 0.00 -> 184.4 mm, vias 0 -> 2
- net m0r5MOS: track 0.00 -> 181.2 mm, vias 0 -> 2
- net m0c7: track 0.00 -> 171.9 mm, vias 0 -> 3
- net col0: track 171.8 -> 0.00 mm, vias 3 -> 0
- net m0c6: track 0.00 -> 157.5 mm, vias 0 -> 2
- net col2: track 145.1 -> 0.00 mm, vias 3 -> 0
- net m0c1: track 0.00 -> 142.3 mm, vias 0 -> 2
- net col1: track 139.7 -> 0.00 mm, vias 3 -> 0
- net row0: track 136.0 -> 0.00 mm
- net row1: track 122.6 -> 0.00 mm, vias 4 -> 0
- net m0c3: track 0.00 -> 121.5 mm, vias 0 -> 2
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Other:
- board size 104 x 83.9 mm -> 323.9 x 95.2 mm
- board text removed: "ParaKeyt Reference r0.7 UMass ECE SDP26 Team 32 Bennett Gilig, Raffi Belorian, Rikhav Shah, Shlok Raval, Theo Krueger. THIS SIDE FACE DOWN"
- board text removed: "^ This (H16) intentionally has a filled zone for interference tests"
