File: test.kicad_pcb (KiCad board)
At the start: 2 copper layers, 285.8 x 95.2 mm, 64 parts

Commit message: adds heuristic
Parts:
- removed the REF** at (21.0, 21.0)
- removed the REF** at (21.0, 32.4)
- added REF**: WQFN16_RTE_TEX_with_caps_and_Rs, WQFN16_RTE_TEX_with_caps_and_Rs, F.Cu at (270.5, 13.3)
- added REF**: WQFN16_RTE_TEX_with_caps_and_Rs, WQFN16_RTE_TEX_with_caps_and_Rs, F.Cu at (270.5, 3.81)
Changed lines of the file:
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@@
   )
   (footprint "WQFN16_RTE_TEX_with_caps_and_Rs" (version 20241229) (generator pcbnew) (layer "F.Cu")
-    (at 20.95500000000001 20.95500000000001)
+    (at 270.50999999999993 13.335000000000004)
     (tags "TLA2528IRTER ")
     (property "Reference" "REF**")
@@
   )
   (footprint "WQFN16_RTE_TEX_with_caps_and_Rs" (version 20241229) (generator pcbnew) (layer "F.Cu")
-    (at 20.95500000000001 32.38500000000001)
+    (at 270.50999999999993 3.8100000000000005)
     (tags "TLA2528IRTER ")
     (property "Reference" "REF**")

Commit message: footprint stuff
Parts:
- removed REF** (x8): SC59_DIO_KeyswitchOutline_NoRuleArea_mosfet, SC59_DIO_KeyswitchOutline_NoRuleArea_mosfet
- removed REF** (x53): SC59_DIO_KeyswitchOutline_NoRuleArea_mosfet, SC59_DIO_KeyswitchOutline_NoRuleArea
- removed REF** (x2): WQFN16_RTE_TEX_with_caps_and_Rs, WQFN16_RTE_TEX_with_caps_and_Rs
- removed U?: rp2040-zero-tht, rp2040-zero-tht
- added R0: rp2040-zero-tht, rp2040-zero-tht, F.Cu at (328.6, 12.0)
- added R1: SC59_DIO_KeyswitchOutline_NoRuleArea_mosfet, SC59_DIO_KeyswitchOutline_NoRuleArea_mosfet, F.Cu at (9.53, 9.53)
- added R10: SC59_DIO_KeyswitchOutline_NoRuleArea_mosfet, SC59_DIO_KeyswitchOutline_NoRuleArea, F.Cu at (181.0, 9.53)
- added R11: SC59_DIO_KeyswitchOutline_NoRuleArea_mosfet, SC59_DIO_KeyswitchOutline_NoRuleArea, F.Cu at (200.0, 9.53)
- added R12: SC59_DIO_KeyswitchOutline_NoRuleArea_mosfet, SC59_DIO_KeyswitchOutline_NoRuleArea, F.Cu at (219.1, 9.53)
- added R13: SC59_DIO_KeyswitchOutline_NoRuleArea_mosfet, SC59_DIO_KeyswitchOutline_NoRuleArea, F.Cu at (238.1, 9.53)
- added R14: SC59_DIO_KeyswitchOutline_NoRuleArea_mosfet, SC59_DIO_KeyswitchOutline_NoRuleArea, F.Cu at (266.7, 9.53)
- added R15: SC59_DIO_KeyswitchOutline_NoRuleArea_mosfet, SC59_DIO_KeyswitchOutline_NoRuleArea, F.Cu at (14.3, 28.6)
- added R16: SC59_DIO_KeyswitchOutline_NoRuleArea_mosfet, SC59_DIO_KeyswitchOutline_NoRuleArea, F.Cu at (38.1, 28.6)
- added R17: SC59_DIO_KeyswitchOutline_NoRuleArea_mosfet, SC59_DIO_KeyswitchOutline_NoRuleArea_mosfet, F.Cu at (57.2, 28.6)
- added R18: SC59_DIO_KeyswitchOutline_NoRuleArea_mosfet, SC59_DIO_KeyswitchOutline_NoRuleArea, F.Cu at (76.2, 28.6)
- added R19: SC59_DIO_KeyswitchOutline_NoRuleArea_mosfet, SC59_DIO_KeyswitchOutline_NoRuleArea, F.Cu at (95.2, 28.6)
- added R2: SC59_DIO_KeyswitchOutline_NoRuleArea_mosfet, SC59_DIO_KeyswitchOutline_NoRuleArea, F.Cu at (28.6, 9.53)
- added R20: SC59_DIO_KeyswitchOutline_NoRuleArea_mosfet, SC59_DIO_KeyswitchOutline_NoRuleArea, F.Cu at (114.3, 28.6)
- added R21: SC59_DIO_KeyswitchOutline_NoRuleArea_mosfet, SC59_DIO_KeyswitchOutline_NoRuleArea, F.Cu at (133.3, 28.6)
- added R22: SC59_DIO_KeyswitchOutline_NoRuleArea_mosfet, SC59_DIO_KeyswitchOutline_NoRuleArea, F.Cu at (152.4, 28.6)
- added R23: SC59_DIO_KeyswitchOutline_NoRuleArea_mosfet, SC59_DIO_KeyswitchOutline_NoRuleArea, F.Cu at (171.5, 28.6)
- added R24: SC59_DIO_KeyswitchOutline_NoRuleArea_mosfet, SC59_DIO_KeyswitchOutline_NoRuleArea, F.Cu at (190.5, 28.6)
- added R25: SC59_DIO_KeyswitchOutline_NoRuleArea_mosfet, SC59_DIO_KeyswitchOutline_NoRuleArea_mosfet, F.Cu at (209.6, 28.6)
- added R26: SC59_DIO_KeyswitchOutline_NoRuleArea_mosfet, SC59_DIO_KeyswitchOutline_NoRuleArea, F.Cu at (228.6, 28.6)
- added R27: SC59_DIO_KeyswitchOutline_NoRuleArea_mosfet, SC59_DIO_KeyswitchOutline_NoRuleArea, F.Cu at (247.7, 28.6)
- added R28: SC59_DIO_KeyswitchOutline_NoRuleArea_mosfet, SC59_DIO_KeyswitchOutline_NoRuleArea, F.Cu at (271.5, 28.6)
- added R29: SC59_DIO_KeyswitchOutline_NoRuleArea_mosfet, SC59_DIO_KeyswitchOutline_NoRuleArea, F.Cu at (16.7, 47.6)
- added R3: SC59_DIO_KeyswitchOutline_NoRuleArea_mosfet, SC59_DIO_KeyswitchOutline_NoRuleArea, F.Cu at (47.6, 9.53)
- added R30: SC59_DIO_KeyswitchOutline_NoRuleArea_mosfet, SC59_DIO_KeyswitchOutline_NoRuleArea, F.Cu at (42.9, 47.6)
- added R31: SC59_DIO_KeyswitchOutline_NoRuleArea_mosfet, SC59_DIO_KeyswitchOutline_NoRuleArea, F.Cu at (61.9, 47.6)
- added R32: SC59_DIO_KeyswitchOutline_NoRuleArea_mosfet, SC59_DIO_KeyswitchOutline_NoRuleArea, F.Cu at (81.0, 47.6)
- added R33: SC59_DIO_KeyswitchOutline_NoRuleArea_mosfet, SC59_DIO_KeyswitchOutline_NoRuleArea_mosfet, F.Cu at (100.0, 47.6)
- added R34: SC59_DIO_KeyswitchOutline_NoRuleArea_mosfet, SC59_DIO_KeyswitchOutline_NoRuleArea, F.Cu at (119.1, 47.6)
- added R35: SC59_DIO_KeyswitchOutline_NoRuleArea_mosfet, SC59_DIO_KeyswitchOutline_NoRuleArea, F.Cu at (138.1, 47.6)
- added R36: SC59_DIO_KeyswitchOutline_NoRuleArea_mosfet, SC59_DIO_KeyswitchOutline_NoRuleArea, F.Cu at (157.2, 47.6)
- added R37: SC59_DIO_KeyswitchOutline_NoRuleArea_mosfet, SC59_DIO_KeyswitchOutline_NoRuleArea, F.Cu at (176.2, 47.6)
- added R38: SC59_DIO_KeyswitchOutline_NoRuleArea_mosfet, SC59_DIO_KeyswitchOutline_NoRuleArea, F.Cu at (195.3, 47.6)
- added R39: SC59_DIO_KeyswitchOutline_NoRuleArea_mosfet, SC59_DIO_KeyswitchOutline_NoRuleArea, F.Cu at (214.3, 47.6)
- added R4: SC59_DIO_KeyswitchOutline_NoRuleArea_mosfet, SC59_DIO_KeyswitchOutline_NoRuleArea, F.Cu at (66.7, 9.53)
- added R40: SC59_DIO_KeyswitchOutline_NoRuleArea_mosfet, SC59_DIO_KeyswitchOutline_NoRuleArea, F.Cu at (233.4, 47.6)
- added R41: SC59_DIO_KeyswitchOutline_NoRuleArea_mosfet, SC59_DIO_KeyswitchOutline_NoRuleArea_mosfet, F.Cu at (264.3, 47.6)
- added R42: SC59_DIO_KeyswitchOutline_NoRuleArea_mosfet, SC59_DIO_KeyswitchOutline_NoRuleArea, F.Cu at (21.4, 66.7)
- added R43: SC59_DIO_KeyswitchOutline_NoRuleArea_mosfet, SC59_DIO_KeyswitchOutline_NoRuleArea, F.Cu at (52.4, 66.7)
- added R44: SC59_DIO_KeyswitchOutline_NoRuleArea_mosfet, SC59_DIO_KeyswitchOutline_NoRuleArea, F.Cu at (71.4, 66.7)
- added R45: SC59_DIO_KeyswitchOutline_NoRuleArea_mosfet, SC59_DIO_KeyswitchOutline_NoRuleArea, F.Cu at (90.5, 66.7)
- added R46: SC59_DIO_KeyswitchOutline_NoRuleArea_mosfet, SC59_DIO_KeyswitchOutline_NoRuleArea, F.Cu at (109.5, 66.7)
- added R47: SC59_DIO_KeyswitchOutline_NoRuleArea_mosfet, SC59_DIO_KeyswitchOutline_NoRuleArea, F.Cu at (128.6, 66.7)
- added R48: SC59_DIO_KeyswitchOutline_NoRuleArea_mosfet, SC59_DIO_KeyswitchOutline_NoRuleArea, F.Cu at (147.6, 66.7)
- added R49: SC59_DIO_KeyswitchOutline_NoRuleArea_mosfet, SC59_DIO_KeyswitchOutline_NoRuleArea_mosfet, F.Cu at (166.7, 66.7)
- added R5: SC59_DIO_KeyswitchOutline_NoRuleArea_mosfet, SC59_DIO_KeyswitchOutline_NoRuleArea, F.Cu at (85.7, 9.53)
- added R50: SC59_DIO_KeyswitchOutline_NoRuleArea_mosfet, SC59_DIO_KeyswitchOutline_NoRuleArea, F.Cu at (185.7, 66.7)
- added R51: SC59_DIO_KeyswitchOutline_NoRuleArea_mosfet, SC59_DIO_KeyswitchOutline_NoRuleArea, F.Cu at (204.8, 66.7)
- added R52: SC59_DIO_KeyswitchOutline_NoRuleArea_mosfet, SC59_DIO_KeyswitchOutline_NoRuleArea, F.Cu at (223.8, 66.7)
- added R53: SC59_DIO_KeyswitchOutline_NoRuleArea_mosfet, SC59_DIO_KeyswitchOutline_NoRuleArea, F.Cu at (250.0, 66.7)
- added R54: SC59_DIO_KeyswitchOutline_NoRuleArea_mosfet, SC59_DIO_KeyswitchOutline_NoRuleArea, F.Cu at (11.9, 85.7)
- added R55: SC59_DIO_KeyswitchOutline_NoRuleArea_mosfet, SC59_DIO_KeyswitchOutline_NoRuleArea, F.Cu at (35.7, 85.7)
- added R56: SC59_DIO_KeyswitchOutline_NoRuleArea_mosfet, SC59_DIO_KeyswitchOutline_NoRuleArea, F.Cu at (59.5, 85.7)
- added R57: SC59_DIO_KeyswitchOutline_NoRuleArea_mosfet, SC59_DIO_KeyswitchOutline_NoRuleArea, F.Cu at (81.0, 85.7)
- added R58: SC59_DIO_KeyswitchOutline_NoRuleArea_mosfet, SC59_DIO_KeyswitchOutline_NoRuleArea, F.Cu at (181.0, 85.7)
- added R59: SC59_DIO_KeyswitchOutline_NoRuleArea_mosfet, SC59_DIO_KeyswitchOutline_NoRuleArea_mosfet, F.Cu at (131.0, 85.7)
- added R6: SC59_DIO_KeyswitchOutline_NoRuleArea_mosfet, SC59_DIO_KeyswitchOutline_NoRuleArea, F.Cu at (104.8, 9.53)
- added R60: SC59_DIO_KeyswitchOutline_NoRuleArea_mosfet, SC59_DIO_KeyswitchOutline_NoRuleArea, F.Cu at (200.0, 85.7)
- added R61: SC59_DIO_KeyswitchOutline_NoRuleArea_mosfet, SC59_DIO_KeyswitchOutline_NoRuleArea, F.Cu at (219.1, 85.7)
- added R62: SC59_DIO_KeyswitchOutline_NoRuleArea_mosfet, SC59_DIO_KeyswitchOutline_NoRuleArea, F.Cu at (238.1, 85.7)
- added R63: SC59_DIO_KeyswitchOutline_NoRuleArea_mosfet, SC59_DIO_KeyswitchOutline_NoRuleArea, F.Cu at (276.2, 66.7)
- added R64: SC59_DIO_KeyswitchOutline_NoRuleArea_mosfet, SC59_DIO_KeyswitchOutline_NoRuleArea, F.Cu at (257.2, 85.7)
- added R65: SC59_DIO_KeyswitchOutline_NoRuleArea_mosfet, SC59_DIO_KeyswitchOutline_NoRuleArea, F.Cu at (276.2, 85.7)
- added R66: SC59_DIO_KeyswitchOutline_NoRuleArea_mosfet, SC59_DIO_KeyswitchOutline_NoRuleArea, F.Cu at (295.3, 85.7)
- added R67: WQFN16_RTE_TEX_with_caps_and_Rs, WQFN16_RTE_TEX_with_caps_and_Rs, F.Cu at (342.9, 11.4)
- added R68: WQFN16_RTE_TEX_with_caps_and_Rs, WQFN16_RTE_TEX_with_caps_and_Rs, F.Cu at (312.4, 11.4)
- added R69: SC59_DIO_KeyswitchOutline_NoRuleArea_mosfet, SC59_DIO_KeyswitchOutline_NoRuleArea_mosfet, F.Cu at (295.3, 47.6)
- added R7: SC59_DIO_KeyswitchOutline_NoRuleArea_mosfet, SC59_DIO_KeyswitchOutline_NoRuleArea, F.Cu at (123.8, 9.53)
- added R70: SC59_DIO_KeyswitchOutline_NoRuleArea_mosfet, SC59_DIO_KeyswitchOutline_NoRuleArea, F.Cu at (295.3, 66.7)
- added R71: SC59_DIO_KeyswitchOutline_NoRuleArea_mosfet, SC59_DIO_KeyswitchOutline_NoRuleArea, F.Cu at (295.3, 9.53)
- added R72: SC59_DIO_KeyswitchOutline_NoRuleArea_mosfet, SC59_DIO_KeyswitchOutline_NoRuleArea, F.Cu at (295.3, 28.6)
- added R73: WQFN16_RTE_TEX_with_caps_and_Rs, WQFN16_RTE_TEX_with_caps_and_Rs, F.Cu at (327.7, 28.6)
- added R74: WQFN16_RTE_TEX_with_caps_and_Rs, WQFN16_RTE_TEX_with_caps_and_Rs, F.Cu at (342.9, 22.9)
- added R8: SC59_DIO_KeyswitchOutline_NoRuleArea_mosfet, SC59_DIO_KeyswitchOutline_NoRuleArea, F.Cu at (142.9, 9.53)
- added R9: SC59_DIO_KeyswitchOutline_NoRuleArea_mosfet, SC59_DIO_KeyswitchOutline_NoRuleArea_mosfet, F.Cu at (161.9, 9.53)
Other:
- board size 285.8 x 95.2 mm -> 1733.5 x 104.8 mm
